File: Rev_NC/jar_light.sch (KiCad schematic (older format))
At the start: 25 parts, among them J1 USB_OTG, J2 ISP_CONN_02X03, J4 JST_BATTERY, J6 LEDPAD+, J7 LEDPAD-, Q1 Si3476DV, U1 LTC4054-4.2, U2 ATTINY84A-MUR, U3 FAN3100c

Commit message: added gitignore
Parts:
- C1, C2, C3: symbol C -> device:C
- D1: symbol D_Schottky -> device:D_Schottky
- D2: symbol LED -> device:LED
- D3: symbol D_Zener -> device:D_Zener
- J1: symbol USB_OTG -> jar_light-rescue:USB_OTG
- J2: symbol CONN_02X03 -> jar_light-rescue:CONN_02X03
- J4: symbol CONN_01X02 -> jar_light-rescue:CONN_01X02
- J6, J7: symbol CONN_01X01 -> jar_light-rescue:CONN_01X01
- L1: symbol L -> device:L
- Q1: symbol Si3476DV -> jar_light-rescue:Si3476DV
- R1, R2, R3, R4, R5, R6, R7, R8, R9: symbol R -> device:R
- U1: symbol LTC4054-4.2 -> jar_light-rescue:LTC4054-4.2
- U2: symbol ATTINY84A-MMH -> jar_light-rescue:ATTINY84A-MMH
- U3: symbol FAN3100c -> jar_light-rescue:FAN3100c
Connections:
- wire segments 93 -> 118
